File: Devices/BarrunCUDA/schematic/schematic.kicad_sch (KiCad schematic)
At the start: 25 parts, among them U1 ESP32-WROOM-32

Commit message: asdfsgfda
Parts:
- added Led_X: 4.7k, symbol Device:R
- added XABARA: SW, symbol Sensor:BME280
Connections:
- net 3.3V: now also Led_X.2
- net GND: now also XABARA.
- net at U1.17: now also XABARA.
- new net: Led_X.1, XABARA.
- new net 5V: U1. (3.3V)
- no-connect marks 13 -> 21
Other:
- added sheet BarrunCUDA Controller - Back (schematic_back.kicad_sch)
- note added: "Commutes manually."
- note added: "On this module the power and I^2C lines enter the power I^2C bus."
- note added: "Some of these pins are connected to the breadboard for structure stability only."
- note added: "To back side ----------->"
- note added: "Volume selector"
- note removed: "Manual commuter"
- moved on the sheet: BITNA, Band_B, Band_G, CHIM, GISELLE, GRAN, KARINA, Led_B, Led_G, Led_R, Light_R, MIRU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
