File: Devices/DGRS6/schematic/schematic.kicad_sch (KiCad schematic)
At the start: 25 parts

Commit message: dafsdg
Parts:
- added 100k: R_int, symbol Device:R
- added TouchSensor: ~, symbol Device:R
- 45k: renamed from 100k; value R_float -> R_int
Connections:
- net at 45k.2, Battery.2 (-), Breaker.3 (E)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: now also 100k.2
- net at Battery.1 (+), Front_left.2 (A), Front_right.2 (A)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: now also TouchSensor.1
- net at 1k.1, Reverse protection.1 (K), Reverse protection1.1 (K): now also 100k.1
- net #INT_power_switch-/: now reaches 45k.1, PowerON.1, Reverse protection1.2 (A), Side2.12 (Pin_8)
- net #I_touch_sensor: now reaches Side2.11 (Pin_9)
- net #I_touch_sensor: now also TouchSensor.2
- net #Q_auto_hold: now reaches Reverse protection.2 (A), Side2.13 (Pin_7)
- net at Breaker.2 (C), Side2.18 (Pin_2): now also TouchSensor.3
Other:
- note added: "#INT_power_switch pull-down"
- note added: "Base current limit"
- note added: "Breaker defloat"
- note added: "OR gate I1"
- note added: "OR gate I2"
- note removed: "#INT_/_power_switch"
- note removed: "#Q_auto_hold"
- note removed: "OR gate"
- moved on the sheet: 45k
